Commit message: Improve robot_sim_description packages
Add sim time parameters to view_robot_gazebo.launch.py nodes.

Resolve warning when visualizing the robot in Gazebo.

Create rviz config file for solely visualizing the URDF. Note, sim time
not required when visualizing the URDF.

Organized URDF files. No functional changes made

URDFs from robot_description and robot_sim_description have been made
more similar to make combining them easier

Update diff_drive_controller.yaml update rates in the robot_bringup package.

File: src/robot_sim_description/urdf/ibex_gazebo.urdf.xacro (robot description, xacro)
@@ -1,21 +1,14 @@
 <?xml version="1.0"?>
-<robot xmlns:xacro="http://www.ros.org/wiki/xacro" name="ibex">
+<robot xmlns:xacro="http://www.ros.org/wiki/xacro" name="ibex_gazebo">
     <gazebo>
-    <plugin filename="gz_ros2_control-system" name="gz_ros2_control::GazeboSimROS2ControlPlugin">
-        <parameters>$(find robot_sim_bringup)/config/diff_drive_controller.yaml</parameters>
-    </plugin>
+        <plugin filename="gz_ros2_control-system" name="gz_ros2_control::GazeboSimROS2ControlPlugin">
+            <parameters>$(find robot_sim_bringup)/config/diff_drive_controller.yaml</parameters>
+        </plugin>
     </gazebo>
-        <gazebo>
+    <gazebo>
         <plugin filename="gz-sim-sensors-system" name="gz::sim::systems::Sensors">
             <render_engine>ogre2</render_engine>
         </plugin>
     </gazebo>
-    <!-- <gazebo>
-        <plugin filename="gz-sim-imu-system" name="gz::sim::systems::Imu">
-        </plugin>
-        <plugin filename="gz-sim-sensors-system" name="gz::sim::systems::Sensors">
-            <render_engine>ogre2</render_engine>
-        </plugin>
-    </gazebo> -->
     <gazebo reference="imu_link">
         <sensor name="imu_sensor" type="imu">
@@ -28,29 +21,29 @@
     <gazebo reference="laser_link">
         <sensor name="lidar" type="gpu_lidar">
-        <always_on>true</always_on>
-        <visualize>true</visualize>
-        <topic>scan</topic>
-        <update_rate>5</update_rate>
-        <gz_frame_id>laser_link</gz_frame_id>
-        <lidar>
-            <scan>
-            <horizontal>
-                <samples>360</samples>
-                <resolution>1.00000</resolution>
-                <min_angle>0.000000</min_angle>
-                <max_angle>6.280000</max_angle>
-            </horizontal>
-            </scan>
-            <range>
-            <min>0.120000</min>
-            <max>12.0</max>
-            <resolution>0.02</resolution>
-            </range>
-            <noise>
-            <type>gaussian</type>
-            <mean>0.0</mean>
-            <stddev>0.01</stddev>
-            </noise>
-        </lidar>
+            <always_on>true</always_on>
+            <visualize>true</visualize>
+            <topic>scan</topic>
+            <update_rate>5</update_rate>
+            <gz_frame_id>laser_link</gz_frame_id>
+            <lidar>
+                <scan>
+                    <horizontal>
+                        <samples>360</samples>
+                        <resolution>1.00000</resolution>
+                        <min_angle>-1.570796</min_angle>
+                        <max_angle>1.570796</max_angle>
+                    </horizontal>
+                </scan>
+                <range>
+                    <min>0.300000</min>
+                    <max>12.0</max>
+                    <resolution>0.02</resolution>
+                </range>
+                <noise>
+                    <type>gaussian</type>
+                    <mean>0.0</mean>
+                    <stddev>0.01</stddev>
+                </noise>
+            </lidar>
         </sensor>
     </gazebo>

File: src/robot_sim_description/urdf/ibex_ros2_control.urdf.xacro (robot description, xacro)
@@ -1,4 +1,4 @@
 <?xml version="1.0"?>
-<robot xmlns:xacro="http://www.ros.org/wiki/xacro" name="ibex">
+<robot xmlns:xacro="http://www.ros.org/wiki/xacro" name="ibex_ros2">
   <ros2_control name="GazeboSimSystem" type="system">
       <hardware>

Commit message: Working autonomy without the corrections

File: src/robot_description/urdf/ibex_core.urdf.xacro (robot description, xacro)
@@ -140,5 +140,5 @@
     <!-- ========================================= -->
     <!-- LiDAR Link and Joint -->
-    <link name="laser_link">
+    <link name="laser">
         <inertial>
             <origin xyz="-0.011945780406062 -0.000381929217680526 -0.0170649378129477" rpy="0 0 0" />
@@ -164,5 +164,5 @@
     <joint name="laser_joint" type="fixed">
         <parent link="base_link" />
-        <child link="laser_link" />
+        <child link="laser" />
         <origin xyz="0.45 0 0.12" rpy="0 0 0" />
     </joint>

File: src/robot_description/urdf/ibex_gazebo.urdf.xacro (robot description, xacro)
@@ -19,5 +19,5 @@
         </sensor>
     </gazebo>
-    <gazebo reference="laser_link">
+    <gazebo reference="laser">
         <sensor name="lidar" type="gpu_lidar">
             <always_on>true</always_on>
@@ -25,5 +25,5 @@
             <topic>scan</topic>
             <update_rate>5</update_rate>
-            <gz_frame_id>laser_link</gz_frame_id>
+            <gz_frame_id>laser</gz_frame_id>
             <lidar>
                 <scan>
